Commit message: turtlebo3_description -> turtlebot_burger_description

File: src/turtlebot3_burger_description/urdf/turtlebot3_burger.urdf (robot description, URDF)
Before this commit: robot turtlebot3_burger, 7 links, 6 joints
Links:
- link ${namespace}base_link: geometry collision box size=0.140 0.140 0.143; visual mesh filename=package://turtlebot3_burger_description/meshes/bases/burger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 scale=0.001 0.001 0.001
- link ${namespace}base_scan: geometry collision cylinder length=0.0315 radius=0.055; visual mesh filename=package://turtlebot3_burger_description/meshes/sensors/lds.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 scale=0.001 0.001 0.001
- link ${namespace}wheel_left_link: geometry collision cylinder length=0.018 radius=0.033; visual mesh filename=package://turtlebot3_burger_description/meshes/wheels/left_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 scale=0.001 0.001 0.001
- link ${namespace}wheel_right_link: geometry collision cylinder length=0.018 radius=0.033; visual mesh filename=package://turtlebot3_burger_description/meshes/wheels/right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 scale=0.001 0.001 0.001
